File: output/KiCad_project/gundamBowtie.kicad_pcb (KiCad board)
At the start: 2 copper layers, 377.5 x 199.5 mm, 155 parts

Commit message: gerbersPt.2
Parts:
- moved _8 7.35 mm to (166.9, 142.2)
- moved S57 7.35 mm to (297.0, 148.7)
- moved S16 7.35 mm to (98.7, 142.2)
- moved _10 7.35 mm to (198.4, 226.8)
- moved S66 7.35 mm to (255.3, 74.2)
- moved S58 7.35 mm to (292.5, 129.2)
- moved S8 7.35 mm to (61.0, 104.1)
- moved D65 7.35 mm to (262.8, 102.2)
- moved D46 7.35 mm to (350.1, 65.4)
- moved D29 7.35 mm to (153.1, 102.2)
- moved S69 7.35 mm to (241.1, 185.1)
- moved D39 7.35 mm to (379.3, 106.1)
- moved S65 7.35 mm to (261.5, 97.4)
- moved D61 7.35 mm to (279.3, 71.7)
- moved _4 7.35 mm to (146.1, 81.1)
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Routing:
- net GP1: track 0.00 -> 893.6 mm, vias 0 -> 2
- net GP2: track 0.00 -> 877.3 mm, vias 0 -> 4
- net GP3: track 0.00 -> 789.9 mm
- net GP4: track 0.00 -> 675.8 mm
- net GP0: track 0.00 -> 674.5 mm
- net GP5: track 0.00 -> 484.9 mm
- net GP22: track 0.00 -> 275.5 mm
- net GP19: track 0.00 -> 256.1 mm
- net GP9: track 26.1 -> 282.0 mm
- net GP18: track 4.32 -> 256.4 mm
- net GP21: track 0.00 -> 249.8 mm
- net GP20: track 0.00 -> 237.4 mm
- net GP10: track 25.9 -> 258.4 mm
- net GP13: track 30.2 -> 258.1 mm
- net GP11: track 25.9 -> 251.8 mm
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